File: pocket-reform-motherboard/pocket-reform-motherboard.kicad_sch (KiCad schematic)
At the start: 434 parts, among them J1 CHARGER, J10 1-2199230-6, J11 Conn_01x33, J12 2199230-5, J13 3-2328724-1, J14 USB_C_Receptacle, J15 CONN_SPK, J16 SAMTEC_TSM-106-02-X-SH-A, J17 POWSW, J18 CONN_HEAD, J2 DM3AT-SF-PEJM5, J20 QWIIC, J3 USB_C_Receptacle, J4 09452812561, J5 SYSCTL, J6 USB_INT1, J7 HDMI_D_1.4, J8 SIM_Card, J9 Conn_01x20, SW1 SW_DIP_x01, SW2 RESET, SW3 RESET, U1 reform2-som-connector, U10 W25Q32JVSS, U11 PCF8523T, U12 AP22615AWU-7, U13 TXS0108EPW, U14 SN74AVC1T45, U15 TPD4E02B04DQA, U16 TPD4E02B04DQA, U17 TPD12S521, U18 TLV320AIC3100, U19 TPD4E02B04DQA, U2 TS3USB30EDGSR, U20 TPD4E02B04DQA, U21 TPD4E02B04DQA, U22 TPD4E02B04DQA, U23 FUSB302BMPX, U24 TXS0108EPW, U25 TUSB8041, U26 TPS542021DDC, U27 TVS2200DRV, U28 LM62460, U29 AP22615AWU-7, U3 LM2830XQMFE/NOPB, U30 TS3USB30EDGSR, U31 TS3USB30EDGSR, U32 AP22615AWU-7, U33 AT24CS02-STUM, U34 PCA9536DP, U35 TMUXHS4446RETR, U36 AP22615AWU-7, U37 TS3USB30EDGSR, U38 CY7C65215-32LTXI, U39 PCA9557PW, U4 TLV75718PDBV, U40 AP22615AWU-7, U5 LM73100RPWR, U6 LM62460, U7 74LVC1G34, U8 RP2040, U9 TPS7A0533PDBZ, Y1 24MHz, Y2 12MHz 12pF, Y3 32.768 kHz

Commit message: mb2.0: snapshot before rev2
Other:
- note added: "BRINGUP: adjust ISET TODO: 6.8k/1A is too tight for SSD in tests. switched to 2.2k on board (3A ~ 9.9W)"
- note added: "DP0"
- note added: "DP1"
- note added: "NOTE: bodged on my MB2"
- note added: "TODO: DP AC on this lane vs DP1"
- note added: "TODO: FIXME: redo to include a 5V switch to USB_VBUS. charger board v2 can't use otg because of the protector chip"
- note added: "TODO: polarity swap issue for DP?"
- note added: "TODO: supply vconn!"
- note added: "TODO: swap pol?"
- note removed: "BRINGUP: adjust ISET"
