File: pocket-reform-motherboard/pocket-reform-motherboard.kicad_sch (KiCad schematic)
At the start: 434 parts, among them J1 CHARGER, J10 1-2199230-6, J11 Conn_01x33, J12 2199230-5, J13 3-2328724-1, J14 USB_C_Receptacle, J15 CONN_SPK, J16 SAMTEC_TSM-106-02-X-SH-A, J17 POWSW, J18 CONN_HEAD, J2 DM3AT-SF-PEJM5, J20 QWIIC, J3 USB_C_Receptacle, J4 09452812561, J5 SYSCTL, J6 USB_INT1, J7 HDMI_D_1.4, J8 SIM_Card, J9 Conn_01x20, SW1 SW_DIP_x01, SW2 RESET, SW3 RESET, U1 reform2-som-connector, U10 W25Q32JVSS, U11 PCF8523T, U12 AP22615AWU-7, U13 TXS0108EPW, U14 SN74AVC1T45, U15 TPD4E02B04DQA, U16 TPD4E02B04DQA, U17 TPD12S521, U18 TLV320AIC3100, U19 TPD4E02B04DQA, U2 TS3USB30EDGSR, U20 TPD4E02B04DQA, U21 TPD4E02B04DQA, U22 TPD4E02B04DQA, U23 FUSB302BMPX, U24 TXS0108EPW, U25 TUSB8041, U26 TPS542021DDC, U27 TVS2200DRV, U28 LM62460, U29 AP22615AWU-7, U3 LM2830XQMFE/NOPB, U30 TS3USB30EDGSR, U31 TS3USB30EDGSR, U32 AP22615AWU-7, U33 AT24CS02-STUM, U34 PCA9536DP, U35 TMUXHS4446RETR, U36 AP22615AWU-7, U37 TS3USB30EDGSR, U38 CY7C65215-32LTXI, U39 PCA9557PW, U4 TLV75718PDBV, U40 AP22615AWU-7, U5 LM73100RPWR, U6 LM62460, U7 74LVC1G34, U8 RP2040, U9 TPS7A0533PDBZ, Y1 24MHz, Y2 12MHz 12pF, Y3 32.768 kHz

Commit message: mainboard: 2.0 R-1 schematic with USB and DP fixes
Parts:
- removed R146, R147: 0, Resistor_SMD:R_0402_1005Metric, symbol Device:R_Small
- added C136, C157, C158: 10uF, Capacitor_SMD:C_0603_1608Metric, symbol Device:C_Small
- added C137, C138: 0.1uF, Capacitor_SMD:C_0402_1005Metric, symbol Device:C_Small
- added R142, R143: 10k, Resistor_SMD:R_0402_1005Metric, symbol Device:R_Small
- added R166, R167, R168, R169, R170: 0, Resistor_SMD:R_0402_1005Metric, symbol Device:R_Small
- added TP20, TP21: TestPoint, symbol Connector:TestPoint
- added U41: AP22615AWU-7, Package_TO_SOT_SMD:SOT-23-6, symbol Regulator_Linear:AP22615AWU
- R150, R157: now fitted
- R158, R32: value 6.8k -> 2.2k
- R33: value 0 -> 2.2k; LCSC C17168 -> C25917; Manufacturer_No 0402WGF0000TCE -> 0402WGF6801TCE
Connections:
- net +5V: now also C136.1, R142.2, U41.6 (IN)
- net DP_AUX_N: now also C138.2
- net DP_AUX_P: now also C137.2
- net GND: now also R33.2, C136.2, C157.2, C158.2, R143.1, U41.2 (GND)
- net MODEM_3V3: now also R166.2
- net USBM2_AC_TXN: now also C91.2; no longer C93.2
- net USBM2_AC_TXP: now also C93.2; no longer C91.2
- net USBM_DP0_N: now also U35.39 (DP0+); no longer U35.40 (DP0-)
- net USBM_DP0_P: now also U35.40 (DP0-); no longer U35.39 (DP0+)
- net USBM_DP1_N: now also U35.2 (DP1+); no longer U35.3 (DP1-)
- net USBM_DP1_P: now also U35.3 (DP1-); no longer U35.2 (DP1+)
- net USBM_DP_AUX_N: now also C138.1
- net USBM_DP_AUX_P: now also C137.1
- net USB_VBUS: now also C157.1, C158.1, U41.1 (OUT)
- net USBM_DP2_N: now reaches U35.5 (DP2+)
- net USBM_DP2_N: now also R169.2
- net USBM_DP2_P: now reaches U35.6 (DP2-)
- net USBM_DP2_P: now also R170.2
- net USBM_DP3_N: now reaches U35.8 (DP3+)
- net USBM_DP3_N: now also R167.2
- net USBM_DP3_P: now reaches U35.9 (DP3-)
- net USBM_DP3_P: now also R168.2
- net USB_SRC2_EN: now reaches U8.41 (GPIO29_ADC3)
- net USB_SRC2_EN: now also R49.2, U12.4 (EN)
- net at J14.A5 (CC1), U15.1 (IO1), U15.10 (IO1)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: now also TP20.1
- net at J14.B5 (CC2), U15.2 (IO2), U15.9 (IO2)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: now also TP21.1
- net at U23.12 (VCONN): now also U23.13 (VCONN), R166.1
- net DP2_P: now reaches J9.1 (Pin_1)
- net DP2_P: now also R170.1
- net DP3_P: now reaches J9.10 (Pin_10)
- net DP3_P: now also R168.1
- net DP3_N: now reaches J9.11 (Pin_11)
- net DP3_N: now also R167.1
- net DP2_N: now reaches J9.2 (Pin_2)
- net DP2_N: now also R169.1
- net R_USB_SRC_EN: no longer names the net of R33.1
- net R_USB_SRC_EN: now also U41.5 (ISET); no longer U8.40 (GPIO28_ADC2)
- removed net USB_SRC_EN: R33.2, R49.2, U12.4 (EN)
- new net: R142.1, U41.3 (FLG)
- new net USB_SRC1_EN: R143.2, U41.4 (EN), U8.40 (GPIO28_ADC2)
- no-connect marks 219 -> 208
Other:
- note added: "2.0 R-1 change"
- note added: "2.0 R-1 change: USB SRC1/2 split"
- note added: "2.0 R-1 change: VCONN. MODEM_3V3 is convenient on the PCB"
- note added: "2.0 R-1 change: include a 5V switch to USB_VBUS. charger board v2 can't use otg because of the protector chip"
- note added: "2.0 R-1: DP1 swapped too, like all others"
- note added: "2.0 R-1: adds lane 2+3"
- note added: "2.0 R-1: polarity swapped to undo the swap on output side"
- note added: "BRINGUP: adjust ISET 2.0 R-1: 6.8k/1A was too tight for SSD in tests. switched to 2.2k on board (3A ~ 9.9W)"
- note added: "CEC"
- note added: "HPD signal for eDP"
- note added: "TODO: AC?"
- note removed: "BRINGUP: adjust ISET TODO: 6.8k/1A is too tight for SSD in tests. switched to 2.2k on board (3A ~ 9.9W)"
- note removed: "LATER: add DP2+DP3"
- note removed: "LATER: any termination needed?"
- note removed: "NOTE: bodged on my MB2"
- note removed: "TODO: FIXME: redo to include a 5V switch to USB_VBUS. charger board v2 can't use otg because of the protector chip"
- note removed: "TODO: polarity swap issue for DP?"
- note removed: "TODO: supply vconn!"
- note removed: "TODO: swap pol?"
- note removed: "on V1: power enables"
- note removed: "there was a diode here in V1.0 pointing towards VCHG. since V1.5, VCHG can also output to the USB-C port (use OTG VBUS function)."
- moved on the sheet: C152, C153, C47, R165, R31, R32, R49, R68, U12, U27

Commit message: mainboard 2.0 r-1 polished
Parts:
- TP20, TP21: footprint (none) -> TestPoint:TestPoint_Pad_D1.0mm
Connections:
- net VCONN: now reaches R166.1, U23.12 (VCONN), U23.13 (VCONN)
Changed lines of the file:
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@@
 		)
 	)
+	(label "VCONN"
+		(at 1101.09 55.88 0)
+		(effects
+			(font
+				(size 1.27 1.27)
+			)
+			(justify left bottom)
+		)
+	)
 	(label "DP3_P"
 		(at 1087.12 270.51 0)
@@
 			)
 		)
-		(property "Footprint" ""
+		(property "Footprint" "TestPoint:TestPoint_Pad_D1.0mm"
 			(at 1036.32 81.28 0)
 			(hide yes)
@@
 			)
 		)
-		(property "Footprint" ""
+		(property "Footprint" "TestPoint:TestPoint_Pad_D1.0mm"
 			(at 1050.29 81.28 0)
 			(hide yes)

Commit message: mb2.0: component updates
Parts:
- C1, C100, C101, C104, C106, C108, C109, C11, C110, C111, C113, C114, C116, C117, C118, C119, C120, C121, C122, C125, C127, C128, C13, C130, C131, C132, C134, C137, C138, C14, C142, C143, C144, C145, C146, C147, C148, C15, C150, C151, C154, C155, C156, C16, C17, C18, C19, C20, C25, C26, C27, C28, C29, C3, C30, C31, C32, C33, C34, C35, C36, C38, C40, C41, C42, C43, C44, C45, C46, C48, C49, C50, C52, C53, C54, C55, C57, C59, C6, C60, C61, C62, C63, C64, C66, C67, C68, C69, C70, C71, C72, C73, C74, C75, C76, C77, C78, C79, C8, C80, C81, C82, C84, C85, C86, C87, C88, C89, C90, C91, C92, C93, C94, C95, C96, C97, C99: Manufacturer Samsung -> (none)
- C10, C102, C103, C123, C124, C126, C135, C22, C24, C83, C9, FB10, FB12, FB13, FB14, FB15, FB16, FB2, FB5, FB9, L1, L2, L5, L6: Manufacturer Murata -> (none)
- C105, C107, C112, C115, C12, C129, C133, C136, C141, C149, C152, C153, C157, C158, C2, C39, C47, C51, C56, C58, C65, C7, C98: Manufacturer muRata -> (none)
- C21, C23, C37: Manufacturer FH -> (none)
- C4: Manufacturer Nichicon -> (none)
- C5: Manufacturer Lelon -> (none)
- D1, D23, D8, D9: Manufacturer XINGLIGHT -> (none)
- D10: Manufacturer Everlight -> (none)
- D12: Manufacturer AVX -> (none)
- D2, U13, U14, U15, U16, U17, U18, U19, U2, U20, U21, U22, U24, U25, U26, U27, U28, U3, U30, U31, U34, U35, U37, U4, U5, U6, U9: Manufacturer Texas Instruments -> (none)
- D3: Manufacturer MSKSEMI -> (none)
- D5: Manufacturer FUXINSEMI -> (none)
- H5, H7, H8, H9: Manufacturer Wurth -> (none)
- J1: Manufacturer HR(Joint Tech Elec) -> (none)
- J10, J12, U1: Manufacturer TE -> (none)
- J11: Manufacturer Yuandi -> (none)
- J13: Manufacturer Guoconn -> (none)
- J14, J15, J3, J8: Manufacturer Molex -> (none)
- J16: Manufacturer Samtec -> (none)
- J17, J18, J20, J5, J6: Manufacturer JST -> (none)
- J2: Manufacturer Hirose -> (none)
- J4: Manufacturer HARTING -> (none)
- J7: Manufacturer Bossie -> (none)
- J9: Manufacturer HCTL -> (none)
- L3, L4: Manufacturer cijang -> (none)
- R1, R10, R100, R101, R102, R103, R104, R105, R106, R107, R108, R109, R11, R110, R111, R112, R113, R114, R115, R116, R117, R118, R119, R12, R120, R121, R122, R123, R124, R125, R126, R127, R128, R129, R13, R130, R131, R132, R133, R134, R135, R136, R137, R138, R139, R14, R140, R141, R142, R143, R144, R145, R148, R149, R15, R150, R151, R152, R153, R154, R155, R156, R157, R159, R16, R160, R161, R162, R163, R164, R165, R166, R167, R168, R169, R17, R170, R18, R19, R198, R199, R2, R20, R22, R23, R24, R25, R26, R27, R28, R29, R3, R30, R31, R34, R35, R36, R37, R38, R39, R4, R40, R41, R42, R43, R44, R45, R46, R47, R48, R49, R5, R50, R51, R52, R53, R54, R56, R57, R58, R59, R6, R60, R61, R62, R63, R64, R65, R66, R67, R68, R69, R7, R70, R71, R72, R73, R75, R76, R77, R79, R80, R81, R82, R83, R84, R85, R87, R89, R9, R90, R91, R92, R93, R94, R95, R96, R97, R98, R99: Manufacturer UNI-ROYAL -> (none)
- R158, R32, R33: LCSC C25917 -> C25879; Manufacturer UNI-ROYAL -> (none); Manufacturer_No 0402WGF6801TCE -> 0402WGF2201TCE
- R21, R74, R78, R88, TP1, TP10, TP11, TP12, TP13, TP14, TP15, TP16, TP17, TP18, TP19, TP2, TP3, TP4, TP5, TP6, TP7, TP8, TP9: Manufacturer DNP -> (none)
- R55, R86: Manufacturer UNI-ROYAL -> (none); now fitted
- SW1: Manufacturer Nidec -> (none)
- SW2, SW3: Manufacturer XKB -> (none)
- TP20, TP21: Manufacturer_No (none) -> DNP; now not fitted
- TR1: Manufacturer Heling -> (none)
- U10: Manufacturer Winbond -> (none)
- U11, U39: Manufacturer NXP -> (none)
- U12, U29, U32, U36, U40, U41: Manufacturer Diodes -> (none)
- U23: Manufacturer ON Semi -> (none)
- U33: Manufacturer Microchip -> (none)
- U38: Manufacturer Infineon -> (none)
- U7: Manufacturer Texas Instruments or UMW -> (none)
- U8: Manufacturer Raspberry Pi -> (none)
- Y1, Y3: Manufacturer Seiko Epson -> (none)
- Y2: Manufacturer Abracon -> (none)
