File: pocket-reform-motherboard/pocket-reform-motherboard.kicad_sch (KiCad schematic)
At the start: 447 parts, among them J1 CHARGER, J10 1-2199230-6, J11 Conn_01x33, J12 2199230-5, J13 3-2328724-1, J14 USB_C_Receptacle, J15 CONN_SPK, J16 SAMTEC_TSM-106-02-X-SH-A, J17 POWSW, J18 CONN_HEAD, J2 DM3AT-SF-PEJM5, J20 QWIIC, J3 USB_C_Receptacle, J4 09452812561, J5 SYSCTL, J6 USB_INT1, J7 HDMI_D_1.4, J8 SIM_Card, J9 Conn_01x20, SW1 SW_DIP_x01, SW2 RESET, SW3 RESET, U1 reform2-som-connector, U10 W25Q32JVSS, U11 PCF8523T, U12 AP22615AWU-7, U13 TXS0108EPW, U14 SN74AVC1T45, U15 TPD4E02B04DQA, U16 TPD4E02B04DQA, U17 TPD12S521, U18 TLV320AIC3100, U19 TPD4E02B04DQA, U2 TS3USB30EDGSR, U20 TPD4E02B04DQA, U21 TPD4E02B04DQA, U22 TPD4E02B04DQA, U23 FUSB302BMPX, U24 TXS0108EPW, U25 TUSB8041, U26 TPS542021DDC, U27 TVS2200DRV, U28 LM62460, U29 AP22615AWU-7, U3 LM2830XQMFE/NOPB, U30 TS3USB30EDGSR, U31 TS3USB30EDGSR, U32 AP22615AWU-7, U33 AT24CS02-STUM, U34 PCA9536DP, U35 TMUXHS4446RETR, U36 AP22615AWU-7, U37 TS3USB30EDGSR, U38 CY7C65215-32LTXI, U39 PCA9557PW, U4 TLV75718PDBV, U40 AP22615AWU-7, U41 AP22615AWU-7, U5 LM73100RPWR, U6 LM62460, U7 74LVC1G34, U8 RP2040, U9 TPS7A0533PDBZ, Y1 24MHz, Y2 12MHz 12pF, Y3 32.768 kHz

Commit message: mb2.0 r-1: last minute 3v3 standby dcdc change
Parts:
- removed C149: 10uF, Capacitor_SMD:C_0603_1608Metric, symbol Device:C_Small
- removed C150: 0.1uF, Capacitor_SMD:C_0402_1005Metric, symbol Device:C_Small
- removed R140: 100k, Resistor_SMD:R_0402_1005Metric, symbol Device:R_Small
- removed R9: 22k, Resistor_SMD:R_0402_1005Metric, symbol Device:R_Small
- removed U26: TPS542021DDC, Package_TO_SOT_SMD:SOT-23-6, symbol Regulator_Switching:TPS54202DDC
- added U42: TPS560430X3FDBVR, Package_TO_SOT_SMD:SOT-23-6, symbol Regulator_Switching:LMR16006YQ3
- L1: value 10uH -> 12uH; footprint Inductor_SMD:L_1210_3225Metric -> Inductor_SMD:L_Taiyo-Yuden_NR-30xx; LCSC C1333678 -> C167758; Manufacturer_No DFE322512F-100M=P2 -> FNR3015S120MT
- R72: value 100k -> 10k; LCSC C25741 -> C25744; Manufacturer_No 0402WGF1003TCE -> 0402WGF1002TCE
Connections:
- net GND: now also U42.2 (GND)
- net SYS_VCC: now also U42.5 (VIN)
- net VCC: now also U42.3 (FB)
- net ~{STANDBY_SHDN}: now also U42.4 (~{SHDN})
- net at C109.1, L1.1: now also U42.6 (SW)
- net at C109.2: now also U42.1 (CB)
Other:
- note added: "4V-36V"
- note removed: "4.5V-30V"
- moved on the sheet: C109, C135, C2
