File: pocket-reform-motherboard/pocket-reform-motherboard.kicad_pcb (KiCad board)
At the start: 6 copper layers, 151 x 88 mm, 434 parts, among them J1 CHARGER, J10 1-2199230-6, J11 Conn_01x33, J12 2199230-5, J13 3-2328724-1, J14 USB_C_Receptacle, J15 CONN_SPK, J16 SAMTEC_TSM-106-02-X-SH-A, J17 POWSW, J18 CONN_HEAD, J2 DM3AT-SF-PEJM5, J20 QWIIC, J3 USB_C_Receptacle, J4 09452812561, J5 SYSCTL, J6 USB_INT1, J7 HDMI_D_1.4, J8 SIM_Card, J9 Conn_01x20, SW1 SW_DIP_x01, SW2 RESET, SW3 RESET, U1 reform2-som-connector, U10 W25Q32JVSS, U11 PCF8523T, U12 AP22615AWU-7, U13 TXS0108EPW, U14 SN74AVC1T45, U15 TPD4E02B04DQA, U16 TPD4E02B04DQA, U17 TPD12S521, U18 TLV320AIC3100, U19 TPD4E02B04DQA, U2 TS3USB30EDGSR, U20 TPD4E02B04DQA, U21 TPD4E02B04DQA, U22 TPD4E02B04DQA, U23 FUSB302BMPX, U24 TXS0108EPW, U25 TUSB8041, U26 TPS542021DDC, U27 TVS2200DRV, U28 LM62460, U29 AP22615AWU-7, U3 LM2830XQMFE/NOPB, U30 TS3USB30EDGSR, U31 TS3USB30EDGSR, U32 AP22615AWU-7, U33 AT24CS02-STUM, U34 PCA9536DP, U35 TMUXHS4446RETR, U36 AP22615AWU-7, U37 TS3USB30EDGSR, U38 CY7C65215-32LTXI, U39 PCA9557PW, U4 TLV75718PDBV, U40 AP22615AWU-7, U5 LM73100RPWR, U6 LM62460, U7 74LVC1G34, U8 RP2040, U9 TPS7A0533PDBZ, Y1 24MHz, Y2 12MHz 12pF, Y3 32.768 kHz

Commit message: mainboard 2.0 r-1 polished
Parts:
- removed R146, R147: 0, Resistor_SMD:R_0402_1005Metric
- added C136: 10uF, Capacitor_SMD:C_0603_1608Metric, F.Cu at (197.8, 151.2)
- added C137: 0.1uF, Capacitor_SMD:C_0402_1005Metric, F.Cu at (165.3, 83.8)
- added C138: 0.1uF, Capacitor_SMD:C_0402_1005Metric, F.Cu at (166.2, 83.8)
- added C157: 10uF, Capacitor_SMD:C_0603_1608Metric, F.Cu at (198.0, 147.5)
- added C158: 10uF, Capacitor_SMD:C_0603_1608Metric, F.Cu at (199.5, 146.1)
- added R142: 10k, Resistor_SMD:R_0402_1005Metric, F.Cu at (196.5, 151.6)
- added R143: 10k, Resistor_SMD:R_0402_1005Metric, F.Cu at (194.4, 151.6)
- added R166: 0, Resistor_SMD:R_0402_1005Metric, F.Cu at (187.8, 139.5)
- added R167: 0, Resistor_SMD:R_0402_1005Metric, F.Cu at (172.3, 82.7)
- added R168: 0, Resistor_SMD:R_0402_1005Metric, F.Cu at (173.3, 82.7)
- added R169: 0, Resistor_SMD:R_0402_1005Metric, F.Cu at (178.1, 82.7)
- added R170: 0, Resistor_SMD:R_0402_1005Metric, F.Cu at (179.0, 82.7)
- added TP20: TestPoint, TestPoint:TestPoint_Pad_D1.0mm, F.Cu at (179.7, 139.2)
- added TP21: TestPoint, TestPoint:TestPoint_Pad_D1.0mm, F.Cu at (179.7, 137.1)
- added U41: AP22615AWU-7, Package_TO_SOT_SMD:SOT-23-6, F.Cu at (195.5, 148.6)
- D1: value LED_MODEM -> LED_RED
- R158, R32: value 6.8k -> 2.2k
- R33: value 0 -> 2.2k
- moved R131 26.1 mm to (166.3, 134.4), turned to 0 degrees
- moved R33 16.7 mm to (195.4, 151.6), turned to -90 degrees
- moved R152 7.07 mm to (177.1, 82.7)
- moved R151 7.07 mm to (176.2, 82.7)
- moved TP16 5.53 mm to (201.5, 151.5)
- moved R31 3.85 mm to (199.5, 149.1)
- moved U27 3.59 mm to (201.6, 148.1), turned to 90 degrees
- moved C132 2.73 mm to (165.0, 100.7), turned to 0 degrees
- moved R144 2.19 mm to (162.2, 100.3)
- moved R148 1.03 mm to (174.2, 82.7)
- moved R149 1.03 mm to (175.2, 82.7)
- moved C39 0.90 mm to (180.5, 76.0)
- moved C154 0.52 mm to (167.4, 99.8)
- moved J6 0.50 mm to (179.3, 70.2)
- moved R62 0.50 mm to (180.3, 74.0)
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Connections:
- C91 pad 2: /USBM2_AC_TXP -> /USBM2_AC_TXN
- C93 pad 2: /USBM2_AC_TXN -> /USBM2_AC_TXP
- J9 pad 1: unconnected-(J9-Pin_1-Pad1) -> /DP2_P
- J9 pad 10: unconnected-(J9-Pin_10-Pad10) -> /DP3_P
- J9 pad 11: unconnected-(J9-Pin_11-Pad11) -> /DP3_N
- J9 pad 2: unconnected-(J9-Pin_2-Pad2) -> /DP2_N
- R33 pad 1: /R_USB_SRC_EN -> Net-(U41-ISET)
- R33 pad 2: USB_SRC_EN -> GND
- R49 pad 2: USB_SRC_EN -> USB_SRC2_EN
- U12 pad 4: USB_SRC_EN -> USB_SRC2_EN
- U23 pad 12: unconnected-(U23-VCONN-Pad12) -> /VCONN
- U23 pad 13: unconnected-(U23-VCONN-Pad13) -> /VCONN
- U35 pad 2: USBM_DP1_P -> USBM_DP1_N
- U35 pad 3: USBM_DP1_N -> USBM_DP1_P
- U35 pad 39: USBM_DP0_P -> USBM_DP0_N
- U35 pad 40: USBM_DP0_N -> USBM_DP0_P
- U35 pad 5: unconnected-(U35-DP2+-Pad5) -> USBM_DP2_N
- U35 pad 6: unconnected-(U35-DP2--Pad6) -> USBM_DP2_P
- U35 pad 8: unconnected-(U35-DP3+-Pad8) -> USBM_DP3_N
- U35 pad 9: unconnected-(U35-DP3--Pad9) -> USBM_DP3_P
- U8 pad 40: /R_USB_SRC_EN -> USB_SRC1_EN
- U8 pad 41: unconnected-(U8-GPIO29_ADC3-Pad41) -> USB_SRC2_EN
Routing:
- net USB_SRC1_EN: track 0.00 -> 193.5 mm, vias 0 -> 6
- net USB_SRC2_EN: track 0.00 -> 167.0 mm, vias 0 -> 4
- net /R_USB_SRC_EN: track 163.6 -> 0.00 mm, vias 4 -> 0
- net +5V: track 366.3 -> 401.0 mm, vias 13 -> 18
- net USBM_DP2_N: track 0.00 -> 28.1 mm, vias 0 -> 2
- net USBM_DP2_P: track 0.00 -> 28.0 mm, vias 0 -> 2
- net USBM_DP3_P: track 0.00 -> 27.9 mm, vias 0 -> 2
- net USBM_DP3_N: track 0.00 -> 26.6 mm, vias 0 -> 2
- net /DP2_P: track 0.00 -> 16.4 mm
- net /DP2_N: track 0.00 -> 15.8 mm
- net /DP3_P: track 0.00 -> 11.3 mm
- net /DP3_N: track 0.00 -> 10.7 mm
- net USBM_DP1_P: track 34.1 -> 25.6 mm
- net /DP1_N: track 5.85 -> 13.7 mm
- net USBM_DP1_N: track 34.1 -> 26.3 mm
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Other:
- board text added: "VBUS"
- board text added: "VBUS2"
- board text removed: "TODO: eth d0 trace fix"
- board text removed: "USB_VBUS"
- board text removed: "USB_VBUS2"
